File: setup.sch (EAGLE design)
At the start: 39 parts, among them K1 CPC1708J, K2 CPC1708J, K3 LY30, K4 LY30

Commit message: added stecker
Parts:
- added JP1, JP2, JP3, JP4, JP5, JP6: (no value), pinhead:PINHD-1X2
- added SV1, SV2: (no value), con-lsta:FE08-1
- added SV3, SV4, SV5, SV6, SV7, SV8: (no value), con-lstb:MA04-1
Connections:
- new net N$18: X++.1, Y++.1
- new net N$19: SV2.6, U$1.10
- new net N$20: SV2.5, U$1.11
- new net N$22: Y++.3, Z--/HOME.3
- new net N$23: SV2.4, U$1.12
- new net N$25: SV4.4, X.A+
- new net N$26: SV4.3, X.A-
- new net N$28: SV4.2, X.B+
- new net N$29: SV4.1, X.B-
- new net N$30: SV5.4, Y.A+
- new net N$31: SV5.3, Y.A-
- new net N$32: SV5.2, Y.B+
- new net N$33: SV5.1, Y.B-
- new net N$34: SV6.4, Z.A+
- new net N$35: SV6.3, Z.A-
- new net N$36: SV6.2, Z.B+
- new net N$37: SV6.1, Z.B-
- new net N$38: JP1.2, LASER.GND
- new net N$39: JP1.1, LASER.VCC
- new net N$40: FRAME.GND, JP4.2
- new net N$41: FAN.GND, JP5.2, LED.GND, PUMP.GND
- new net N$42: FAN.VCC, JP5.1, LED.VCC, PUMP.VCC
- net 12V_PC: now also JP6.1; no longer FAN.VCC, LED.VCC, PUMP.VCC
- net 12V_PC_1: now also JP2.1; no longer LASER.VCC
- net COMMON_LIMIT: now also SV1.3, SV2.3; no longer Y++.3, Z--/HOME.3
- net GND_M: now also JP3.2, JP6.2, SV1.8, SV2.8; no longer FAN.GND, FRAME.GND, LED.GND, PUMP.GND, X++.1, Y++.1
- net N$1: now also SV3.4; no longer X.A+
- net N$10: now also SV8.2; no longer Z.B+
- net N$11: now also SV8.1; no longer Z.B-
- net N$12: now also SV7.1; no longer Y.B-
- net N$16: now also JP2.2; no longer LASER.GND
- net N$2: now also SV3.3; no longer X.A-
- net N$3: now also SV3.2; no longer X.B+
- net N$4: now also SV3.1; no longer X.B-
- net N$5: now also SV7.4; no longer Y.A+
- net N$6: now also SV7.3; no longer Y.A-
- net N$7: now also SV7.2; no longer Y.B+
- net N$8: now also SV8.4; no longer Z.A+
- net N$9: now also SV8.3; no longer Z.A-
- net X--/HOME: now also SV1.6; no longer U$1.10
- net Y--/HOME: now also SV1.5; no longer U$1.11
- net Z++/HOME: now also SV1.4; no longer U$1.12
Other:
- note added: "N.C."
- note removed: "some PCB"
- moved on the sheet: LASER, U$4

Commit message: added connectors
Parts:
- added 12V_PC, 12V_PC1, 12V_PC2, 12V_PC3, 36V, 36V1, 36V2, 36V3, L, L1, L10, L11, L13, L14, L15, L16, L17, L18, L19, L2, L20, L21, L23, L24, L25, L26, L3, L4, L5, L6, L7, L8, L9, U$10, U$11, U$5, U$6, U$9: SINGLE_CONNECTOR, libliblib:SINGLE_CONNECTOR
- added GND_MACH: CONNECTOR, libliblib:CONNECTOR
Connections:
- new net 12V_PC_2: 12V_PC.P$11, K34.S
- new net 12V_PC_3: 12V_1.VCC, 12V_PC2.P$11
- new net 12V_PC_4: 12V_PC3.P$11, LED1.C, LED2.C
- new net EAR_1: A_STECKDOSE_PC.EAR, L17.P$11
- new net EAR_2: 5V_1.EAR, I_STECKDOSE.EAR, L16.P$11
- new net EAR_3: 12V_1.EAR, L15.P$11
- new net EAR_4: 5V_M.EAR, L14.P$11
- new net EAR_5: 36V_M.EAR, L13.P$11
- new net GND_M_0: 36V_M.GND, GND_MACH.P$20
- new net GND_M_1: 5V_M.GND, GND_MACH.P$19
- new net GND_M_10: GND_MACH.P$1, SV2.8
- new net GND_M_11: GND_MACH.P$10, JP6.2
- new net GND_M_2: GND_MACH.P$18, MACHINE.1
- new net GND_M_3: GND_MACH.P$16, LED1.A
- new net GND_M_4: 12V_1.GND, GND_MACH.P$17
- new net GND_M_5: GND_MACH.P$14, JP3.2
- new net GND_M_6: GND_MACH.P$13, X.EN-, X.GND
- new net GND_M_7: GND_MACH.P$12, Y.EN-, Y.GND
- new net GND_M_8: GND_MACH.P$11, Z.EN-, Z.GND
- new net GND_M_9: GND_MACH.P$15, U$1.18G, U$1.19G, U$1.20G, U$1.21G, U$1.22G, U$1.23G, U$1.24G, U$1.25G, U$1.S_GND, U$4.S
- new net L1_1: 12V_1.L, L2.P$11
- new net L1_2: 5V_1.L, I_STECKDOSE.L, L3.P$11
- new net L1_3: L4.P$11, PC_ON.3
- new net N$43: L10.P$11, PC_ON.1
- new net N$44: K32.S, L9.P$11
- new net N$45: K33.S, L8.P$11
- new net N$46: K2.DS1, L5.P$11
- new net N$47: 12V_PC.P$1, 12V_PC1.P$1, 12V_PC2.P$1, 12V_PC3.P$1
- new net N$48: K42.P, L6.P$11
- new net N$49: L1.P$1, L2.P$1, L3.P$1, L4.P$1
- new net N$50: 36V.P$1, 36V1.P$1, 36V2.P$1, 36V3.P$1
- new net N$51: 36V1.P$11, Z.VCC
- new net N$52: 36V2.P$11, Y.VCC
- new net N$53: 36V3.P$11, X.VCC
- new net N$54: 5V_M.VCC, U$5.P$11
- new net N$55: K1.K, U$6.P$11
- new net N$56: K2.K, U$9.P$11
- new net N$57: U$10.P$1, U$11.P$1, U$5.P$1, U$6.P$1, U$9.P$1
- new net N$58: A_STECKDOSE_VPUMP.EAR, L14.P$1
- new net N$59: U$1.S_VCC, U$11.P$11
- new net N$60: A_STECKDOSE_VAC.EAR, L13.P$1
- new net N$61: A_STECKDOSE_VPUMP.N, L19.P$1
- new net N$62: A_STECKDOSE_VAC.N, L25.P$1
- new net N$63: L26.P$1, VFD.N
- new net N_1: K31.2, L24.P$11
- new net N_2: K41.2, L23.P$11
- new net N_4: A_STECKDOSE_PC.N, L21.P$11
- new net N_5: 5V_1.N, I_STECKDOSE.N, L20.P$11
- new net N_6: 12V_1.N, L19.P$11
- new net N_7: 5V_M.N, L25.P$11
- new net N_8: 36V_M.N, L26.P$11
- net 12V_PC: now also 12V_PC1.P$11; no longer 12V_1.VCC, K34.S, LED1.C, LED2.C
- net 36V: now also 36V.P$11; no longer X.VCC, Y.VCC, Z.VCC
- net 5V_M: now also U$10.P$11; no longer 5V_M.VCC, K1.K, K2.K, U$1.S_VCC
- net EAR: now also L11.P$11, L15.P$1; no longer 12V_1.EAR, 36V_M.EAR, 5V_1.EAR, 5V_M.EAR, A_STECKDOSE_PC.EAR, A_STECKDOSE_VAC.EAR, A_STECKDOSE_VPUMP.EAR, I_STECKDOSE.EAR
- net GND_M: no longer 12V_1.GND, 36V_M.GND, 5V_M.GND, JP3.2, JP6.2, LED1.A, MACHINE.1, SV2.8, U$1.18G, U$1.19G, U$1.20G, U$1.21G, U$1.22G, U$1.23G, U$1.24G, U$1.25G, U$1.S_GND, U$4.S, X.EN-, X.GND, Y.EN-, Y.GND, Z.EN-, Z.GND
- net L: now also L.P$11, L7.P$11; no longer K2.DS1, K32.S, K33.S, K42.P, PC_ON.1
- net L1: now also L1.P$11; no longer 12V_1.L, 5V_1.L, I_STECKDOSE.L, PC_ON.3
- net N: now also L18.P$11; no longer 12V_1.N, 36V_M.N, 5V_1.N, 5V_M.N, A_STECKDOSE_PC.N, A_STECKDOSE_VAC.N, A_STECKDOSE_VPUMP.N, I_STECKDOSE.N, K31.2, K41.2, VFD.N
Other:
- note added: "10x"
- note added: "12V"
- note added: "36V"
- note added: "4x"
- note added: "5V"
- note added: "5x"
- note added: "6x"
- note added: "7x"
- note added: "8x"
- note added: "=48x"
- note added: "EAR"
- note added: "GND"
- note added: "L"
- note added: "L'"
- note added: "N"
- moved on the sheet: 12V_1, 36V_M, 5V_1, 5V_M, A_STECKDOSE_PC, A_STECKDOSE_VAC, A_STECKDOSE_VPUMP, FAN, FRAME, I_STECKDOSE, JP1, JP2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

Commit message: reality check
Parts:
- removed 5V_M: PWR, libliblib:PWR
- removed I_STECKDOSE: 230VDEV, libliblib:230VDEV
- removed K1: CPC1708J, relay:CPC1708J
- removed K3: LY30, relay:LY30
- removed U$4: N-CHANNEL-MOSFET-BSS138, GeekAmmo:N-CHANNEL-MOSFET-BSS138
- added 5V_M1: PWR, libliblib:PWR
- added K5: CPC1708J, relay:CPC1708J
- added K6: LY30, relay:LY30
- added U$12: N-CHANNEL-MOSFET-BSS138, GeekAmmo:N-CHANNEL-MOSFET-BSS138
Connections:
- net 36V renamed 36V_0
- net N$43 renamed L_1
- net N$51 renamed 36V_1
- net N$52 renamed 36V_2
- net N$53 renamed 36V_3
- net N$59 renamed 5V_M_1
- removed net 5V_M: U$10.P$11, X.DIR+, X.EN+, X.PUL+, Y.DIR+, Y.EN+, Y.PUL+, Z.DIR+, Z.EN+, Z.PUL+
- removed net EAR_2: 5V_1.EAR, I_STECKDOSE.EAR, L16.P$11
- removed net L2: K1.DS2, K2.DS2, K31.1, K41.1
- removed net N$13: U$1.17
- removed net N$19: SV2.6, U$1.10
- removed net N$20: SV2.5, U$1.11
- removed net N$23: SV2.4, U$1.12
- removed net N$24: U$1.6
- removed net N$27: U$1.3
- removed net N$45: K33.S, L8.P$11
- removed net N$48: K42.P, L6.P$11
- removed net N$54: 5V_M.VCC, U$5.P$11
- removed net N$55: K1.K, U$6.P$11
- removed net N$56: K2.K, U$9.P$11
- removed net N_7: 5V_M.N, L25.P$11
- new net 5V_M_0: U$10.P$11, X.DIR+, X.PUL+, Y.DIR+, Y.PUL+, Z.DIR+, Z.PUL+
- new net 5V_M_2: K5.A, U$9.P$11
- new net 5V_M_3: K2.K, U$6.P$11
- new net 5V_M_4: 5V_M1.VCC, U$5.P$11
- new net L_2: K42.P, L9.P$11
- new net L_3: K43.P, L8.P$11
- new net L_4: K2.DS1, L7.P$11
- new net L_5: K64.O, L6.P$11
- new net L_6: K61.1, L5.P$11
- new net N$43: K5.DS2, K61.2
- new net PC_OUT_14: K5.K, U$1.14
- net 12V_PC_1: now also K44.O, LED2.C; no longer K34.P
- net 12V_PC_2: now also K44.P; no longer K34.S
- net 12V_PC_4: no longer LED2.C
- net 5V_PC: no longer U$2.P2
- net EAR_4: now also 5V_M1.EAR; no longer 5V_M.EAR
- net GND_M': now also K2.A; no longer K1.A, LED2.A
- net GND_M_1: now also 5V_M1.GND; no longer 5V_M.GND
- net GND_M_2: now also LED2.A
- net GND_M_9: now also GND_MACH.P$2, U$12.S; no longer U$4.S
- net GND_PC: no longer U$2.N2
- net L: no longer K1.DS1, L7.P$11
- net L1: now also 5V_M1.L
- net L1_2: no longer I_STECKDOSE.L
- net L3: now also K43.S; no longer K33.P
- net L4: now also K42.O; no longer 5V_M.L, K32.P
- net L5: now also K64.P; no longer K42.S
- net LASER_PWM: now also U$1.17, U$12.G; no longer U$1.9, U$4.G
- net N$16: now also U$12.D; no longer U$4.D
- net N$17: now also 5V_M1.N, L23.P$11; no longer K2.A, U$1.14
- net N$44: now also 5V_1.EAR; no longer K32.S, L9.P$11
- net N$46: now also K2.DS2, K41.2; no longer K2.DS1, L5.P$11
- net N_1: now also K41.1; no longer K31.2
- net N_2: now also K5.DS1, L25.P$11; no longer K41.2, L23.P$11
- net N_5: no longer I_STECKDOSE.N
- net X--/HOME: now also SV2.6, U$1.10
- net X_DIR: now also U$1.4; no longer U$1.2
- net X_PUL: now also U$1.5; no longer U$1.1
- net Y--/HOME: now also SV2.5, U$1.11
- net Y_DIR: now also U$1.2; no longer U$1.5
- net Y_PUL: now also U$1.3; no longer U$1.4
- net Z++/HOME: now also SV2.4, U$1.12
- net Z_DIR: now also U$1.6; no longer U$1.8
Other:
- moved on the sheet: 12V_1, 12V_PC, 12V_PC1, 12V_PC2, 12V_PC3, 36V, 36V1, 36V2, 36V3, 36V_M, 5V_1, A_STECKDOSE_VAC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

Commit message: added pendant|
Parts:
- removed MC: LV_DEV, libliblib:LV_DEV
- added U$13: PENDANT, libliblib:PENDANT
- added U$4: POKEY57U, libliblib:POKEY57U
Connections:
- removed net 12V_PC_2: 12V_PC.P$11, K44.P
- removed net 12V_PC_3: 12V_1.VCC, 12V_PC2.P$11
- removed net 12V_PC_4: 12V_PC3.P$11, LED1.C
- removed net 36V_0: 36V.P$11, 36V_M.VCC
- removed net 36V_1: 36V1.P$11, Z.VCC
- removed net 36V_2: 36V2.P$11, Y.VCC
- removed net 36V_3: 36V3.P$11, X.VCC
- removed net 5V_M_0: U$10.P$11, X.DIR+, X.PUL+, Y.DIR+, Y.PUL+, Z.DIR+, Z.PUL+
- removed net 5V_M_1: U$1.S_VCC, U$11.P$11
- removed net 5V_M_2: K5.A, U$9.P$11
- removed net 5V_M_3: K2.K, U$6.P$11
- removed net 5V_M_4: 5V_M1.VCC, U$5.P$11
- removed net EAR_1: A_STECKDOSE_PC.EAR, L17.P$11
- removed net EAR_3: 12V_1.EAR, L15.P$11
- removed net EAR_4: 5V_M1.EAR, L14.P$11
- removed net EAR_5: 36V_M.EAR, L13.P$11
- removed net GND_M_0: 36V_M.GND, GND_MACH.P$20
- removed net GND_M_1: 5V_M1.GND, GND_MACH.P$19
- removed net GND_M_10: GND_MACH.P$1, SV2.8
- removed net GND_M_11: GND_MACH.P$10, JP6.2
- removed net GND_M_2: GND_MACH.P$18, LED2.A, MACHINE.1
- removed net GND_M_3: GND_MACH.P$16, LED1.A
- removed net GND_M_4: 12V_1.GND, GND_MACH.P$17
- removed net GND_M_5: GND_MACH.P$14, JP3.2
- removed net GND_M_6: GND_MACH.P$13, X.EN-, X.GND
- removed net GND_M_7: GND_MACH.P$12, Y.EN-, Y.GND
- removed net GND_M_8: GND_MACH.P$11, Z.EN-, Z.GND
- removed net L1_1: 12V_1.L, L2.P$11
- removed net L1_2: 5V_1.L, L3.P$11
- removed net L1_3: L4.P$11, PC_ON.3
- removed net L3: A_STECKDOSE_VAC.L, K43.S, VFD.L
- removed net L4: 36V_M.L, K42.O
- removed net L_1: L10.P$11, PC_ON.1
- removed net L_2: K42.P, L9.P$11
- removed net L_3: K43.P, L8.P$11
- removed net L_4: K2.DS1, L7.P$11
- removed net L_5: K64.O, L6.P$11
- removed net L_6: K61.1, L5.P$11
- removed net N$17: 5V_M1.N, L23.P$11
- removed net N$58: A_STECKDOSE_VPUMP.EAR, L14.P$1
- removed net N$60: A_STECKDOSE_VAC.EAR, L13.P$1
- removed net N$61: A_STECKDOSE_VPUMP.N, L19.P$1
- removed net N$62: A_STECKDOSE_VAC.N, L25.P$1
- removed net N$63: L26.P$1, VFD.N
- removed net N_1: K41.1, L24.P$11
- removed net N_2: K5.DS1, L25.P$11
- removed net N_4: A_STECKDOSE_PC.N, L21.P$11
- removed net N_5: 5V_1.N, L20.P$11
- removed net N_6: 12V_1.N, L19.P$11
- removed net N_8: 36V_M.N, L26.P$11
- new net 36V: 36V.P$11, 36V1.P$11, 36V2.P$11, 36V3.P$11, 36V_M.VCC, X.VCC, Y.VCC, Z.VCC
- new net 5V_M: 5V_M1.VCC, K2.K, K5.A, U$1.S_VCC, U$10.P$11, U$11.P$11, U$5.P$11, U$6.P$11, U$9.P$11, X.DIR+, X.PUL+, Y.DIR+, Y.PUL+, Z.DIR+, Z.PUL+
- new net L2: 36V_M.L, A_STECKDOSE_VAC.L, K42.O, K43.S, VFD.L
- new net N$13: U$1.1
- new net N$19: U$1.17_PC, U$4.P$22
- new net N$20: U$1.02_PC, U$4.P$39
- new net N$23: U$1.04_PC, U$4.P$38
- new net N$24: U$1.05_PC, U$4.P$46
- new net N$27: U$1.06_PC, U$4.P$40
- new net N$45: U$1.07_PC, U$4.P$49
- new net N$48: U$13.COM, U$13.GND, U$4.GND
- new net N$51: U$13.VCC, U$4.VCC
- new net N$52: U$13.A, U$4.P$1
- new net N$53: U$13.B, U$4.P$2
- new net N$54: U$13.100X
- new net N$55: U$13.10X
- new net N$56: U$13.1X
- new net N$64: U$13.X
- new net N$65: U$13.Y
- new net N$66: U$13.Z
- new net N$67: U$13.C
- new net N$68: U$13.E-STOP
- net 12V_PC: now also 12V_1.VCC, 12V_PC.P$11, 12V_PC2.P$11, 12V_PC3.P$11, K44.P, LED1.C
- net 5V_PC: now also U$4.USB; no longer MC.VCC
- net EAR: now also 12V_1.EAR, 36V_M.EAR, 5V_M1.EAR, A_STECKDOSE_PC.EAR, A_STECKDOSE_VAC.EAR, A_STECKDOSE_VPUMP.EAR, L13.P$1, L13.P$11, L14.P$1, L14.P$11, L15.P$11, L17.P$11
- net GND_M: now also 12V_1.GND, 36V_M.GND, 5V_M1.GND, GND_MACH.P$1, GND_MACH.P$10, GND_MACH.P$11, GND_MACH.P$12, GND_MACH.P$13, GND_MACH.P$14, GND_MACH.P$15, GND_MACH.P$16, GND_MACH.P$17, GND_MACH.P$18, GND_MACH.P$19, GND_MACH.P$20, JP3.2, JP6.2, LED1.A, LED2.A, MACHINE.1, SV2.8, U$1.18G, U$1.19G, U$1.20G, U$1.21G, U$1.22G, U$1.23G, U$1.24G, U$1.25G, U$1.S_GND, X.EN-, X.GND, Y.EN-, Y.GND, Z.EN-, Z.GND
- net GND_M_9: no longer GND_MACH.P$15, U$1.18G, U$1.19G, U$1.20G, U$1.21G, U$1.22G, U$1.23G, U$1.24G, U$1.25G, U$1.S_GND
- net GND_PC: no longer MC.GND, U$2.N1
- net L: now also K2.DS1, K42.P, K43.P, K61.1, K64.O, L10.P$11, L5.P$11, L6.P$11, L7.P$11, L8.P$11, L9.P$11, PC_ON.1
- net L1: now also 12V_1.L, 5V_1.L, L2.P$11, L3.P$11, L4.P$11, PC_ON.3
- net N: now also 12V_1.N, 36V_M.N, 5V_1.N, 5V_M1.N, A_STECKDOSE_PC.N, A_STECKDOSE_VAC.N, A_STECKDOSE_VPUMP.N, K41.1, K5.DS1, L19.P$1, L19.P$11, L20.P$11, L21.P$11, L23.P$11, L24.P$11, L25.P$1, L25.P$11, L26.P$1, L26.P$11, VFD.N
- net N$15: now also U$1.03_PC, U$4.P$48; no longer U$1.PC
Other:
- moved on the sheet: 12V_1, 36V_M, U$12
